Commit message: added gazebo plugin

File: jaguar_description/urdf/accessories/zed.urdf.xacro (robot description, xacro)
@@ -16,5 +16,5 @@
 -->
 <robot name="depth_camera" xmlns:xacro="http://ros.org/wiki/xacro">
-    <xacro:macro name="depth_camera" params="prefix:=depth_camera">
+    <xacro:macro name="depth_camera" params="prefix:=camera">
     <link name="zed_left_camera">
         <visual>
@@ -66,4 +66,48 @@
         <origin xyz="0 -0.06 0" rpy="0 0 0" />
     </joint>
+    <joint name="${prefix}_optical_joint" type="fixed">
+      <origin xyz="0 0 0" rpy="-1.5708 0 -1.5708"/>
+      <parent link="${prefix}_link"/>
+      <child link="${prefix}_frame_optical"/>
+    </joint>
+    <link name="${prefix}_frame_optical"/>
+    <gazebo reference="${prefix}_link">
+      <sensor type="depth" name="${prefix}">
+        <always_on>true</always_on>
+        <update_rate>20.0</update_rate>
+        <camera>
+          <horizontal_fov>${60.0*M_PI/180.0}</horizontal_fov>
+          <image>
+            <format>R8G8B8</format>
+            <width>640</width>
+            <height>480</height>
+          </image>
+          <clip>
+            <near>0.05</near>
+            <far>8.0</far>
+          </clip>
+        </camera>
+        <plugin name="${prefix}_controller" filename="libgazebo_ros_openni_kinect.so">
+          <cameraName>${prefix}</cameraName>
+          <alwaysOn>true</alwaysOn>
+          <updateRate>10</updateRate>
+<!--          <cameraName>${prefix}_ir</cameraName>  -->
+          <imageTopicName>rgb/image_raw</imageTopicName>
+          <depthImageTopicName>depth/image_raw</depthImageTopicName>
+          <pointCloudTopicName>depth/points</pointCloudTopicName>
+          <cameraInfoTopicName>rgb/camera_info</cameraInfoTopicName>
+          <depthImageCameraInfoTopicName>depth/camera_info</depthImageCameraInfoTopicName>
+          <frameName>${prefix}_frame_optical</frameName>
+          <baseline>0.1</baseline>
+          <distortion_k1>0.0</distortion_k1>
+          <distortion_k2>0.0</distortion_k2>
+          <distortion_k3>0.0</distortion_k3>
+          <distortion_t1>0.0</distortion_t1>
+          <distortion_t2>0.0</distortion_t2>
+          <pointCloudCutoff>0.4</pointCloudCutoff>
+          <robotNamespace>/</robotNamespace>
+        </plugin>
+      </sensor>
+    </gazebo>
 </xacro:macro>
 </robot>
