Commit message: minor description fixes

File: jaguar_description/urdf/jaguar.urdf.xacro (robot description, xacro)
@@ -5,5 +5,5 @@
     <property name="M_PI" value="3.14159"/>
     <!-- Wheel Properties -->
-    <xacro:property name="wheel_length" value="0.09"/>
+    <xacro:property name="wheel_length" value="0.085"/>
     <xacro:property name="wheel_radius" value="0.13"/>
     <!-- Base Size -->
@@ -11,6 +11,6 @@
     <property name="wheel_base_offset" value="0.03"/>
     <property name="base_x_size" value="${0.615-2*wheel_base_offset}"/>
-    <property name="base_y_size" value="${0.573-wheel_length}"/>
-    <property name="base_z_size" value="${0.265-distance_from_ground}"/>
+    <property name="base_y_size" value="${0.56-wheel_length}"/>
+    <property name="base_z_size" value="${0.255-distance_from_ground}"/>
     <!-- Wheel Mounting Positions -->
     <xacro:property name="wheelbase" value="${base_x_size-2*wheel_radius+2*wheel_base_offset}"/>
@@ -20,5 +20,5 @@
     <property name="laser_x" value="${base_x_size/2-0.0725}"/>
     <property name="laser_y" value="0"/>
-    <property name="laser_z" value="${0.265+0.05}"/>
+    <property name="laser_z" value="${0.255+0.05}"/>
     <!-- Laser Size -->
     <property name="laser_x_size" value="0.065"/>

Commit message: Added depth camera to robot description

File: jaguar_description/urdf/jaguar.urdf.xacro (robot description, xacro)
@@ -3,4 +3,5 @@
     <!-- Included URDF/XACRO Files -->
     <xacro:include filename="$(find jaguar_description)/urdf/wheel.urdf.xacro"/>
+    <xacro:include filename="$(find jaguar_description)/urdf/accessories/3D_camera.urdf.xacro"/>
     <property name="M_PI" value="3.14159"/>
     <!-- Wheel Properties -->
@@ -136,3 +137,11 @@
     </joint>
     <link name="gps_link"/>
+    <xacro:if value="$(arg 3D_enabled)">
+      <joint name="depth_camera_frame_joint" type="fixed">
+        <origin xyz="0 0 0.525" rpy="0 0 3.14" />
+        <parent link="base_link"/>
+        <child link="depth_camera_link"/>
+      </joint>
+      <xacro:depth_camera prefix="depth_camera"/>
+</xacro:if>
 </robot>

Commit message: webcamera

File: jaguar_description/urdf/jaguar.urdf.xacro (robot description, xacro)
@@ -111,7 +111,7 @@
         <origin xyz="${camera_x} ${camera_y} ${camera_z}" rpy="0 0 0"/>
         <parent link="base_link"/>
-        <child link="camera_link"/>
+        <child link="webcamera_link"/>
     </joint>
-    <link name="camera_link">
+    <link name="webcamera_link">
         <visual>
             <origin xyz="0 0 0" rpy="0 ${M_PI/2} 0"/>
@@ -138,10 +138,10 @@
     <link name="gps_link"/>
     <xacro:if value="$(arg 3D_enabled)">
-      <joint name="depth_camera_frame_joint" type="fixed">
-        <origin xyz="0 0 0.525" rpy="0 0 3.14" />
+      <joint name="camera_frame_joint" type="fixed">
+        <origin xyz="0 0 0.525" rpy="0 0 0 "/>
         <parent link="base_link"/>
-        <child link="depth_camera_link"/>
+        <child link="camera_link"/>
       </joint>
-      <xacro:depth_camera prefix="depth_camera"/>
-</xacro:if>
+      <xacro:depth_camera prefix="camera"/>
+    </xacro:if>
 </robot>

Commit message: Added gazebo plugin

File: jaguar_description/urdf/jaguar.urdf.xacro (robot description, xacro)
@@ -53,5 +53,5 @@
     </link>
     <!-- Interial link stores the robot's inertial information -->
-    <!--<link name="inertial_link">
+    <link name="inertial_link">
         <inertial>
             <mass value="33.455"/>
@@ -64,5 +64,5 @@
         <parent link="base_link"/>
         <child link="inertial_link"/>
-    </joint> -->
+    </joint>
     <!-- IMU exact position is unnecessary thus placed at the center of the platform.-->
     <link name="imu_link"/>
@@ -146,3 +146,37 @@
       <xacro:depth_camera prefix="camera"/>
     </xacro:if>
+      <gazebo>
+    <plugin name="gazebo_ros_control" filename="libgazebo_ros_control.so">
+      <robotNamespace>/</robotNamespace>
+    </plugin>
+  </gazebo>
+  <gazebo>
+    <plugin name="imu_controller" filename="libhector_gazebo_ros_imu.so">
+      <robotNamespace>/</robotNamespace>
+      <updateRate>50.0</updateRate>
+      <bodyName>base_link</bodyName>
+      <topicName>imu/data</topicName>
+      <accelDrift>0.005 0.005 0.005</accelDrift>
+      <accelGaussianNoise>0.005 0.005 0.005</accelGaussianNoise>
+      <rateDrift>0.005 0.005 0.005 </rateDrift>
+      <rateGaussianNoise>0.005 0.005 0.005 </rateGaussianNoise>
+      <headingDrift>0.005</headingDrift>
+      <headingGaussianNoise>0.005</headingGaussianNoise>
+    </plugin>
+  </gazebo>
+  <gazebo>
+    <plugin name="gps_controller" filename="libhector_gazebo_ros_gps.so">
+      <robotNamespace>/</robotNamespace>
+      <updateRate>40</updateRate>
+      <bodyName>base_link</bodyName>
+      <frameId>base_link</frameId>
+      <topicName>navsat/fix</topicName>
+      <velocityTopicName>navsat/vel</velocityTopicName>
+      <referenceLatitude>49.9</referenceLatitude>
+      <referenceLongitude>8.9</referenceLongitude>
+      <referenceHeading>0</referenceHeading>
+      <referenceAltitude>0</referenceAltitude>
+      <drift>0.0001 0.0001 0.0001</drift>
+    </plugin>
+  </gazebo>
 </robot>

Commit message: changed rpyat wheels

File: jaguar_description/urdf/jaguar.urdf.xacro (robot description, xacro)
@@ -77,5 +77,5 @@
     </xacro:jaguar_wheel>
     <xacro:jaguar_wheel wheel_prefix="front_right">
-        <origin xyz="${wheelbase/2} ${-track/2} ${wheel_vertical_offset}" rpy="0 0 ${M_PI}"/>
+        <origin xyz="${wheelbase/2} ${-track/2} ${wheel_vertical_offset}" rpy="0 0 0"/>
     </xacro:jaguar_wheel>
     <xacro:jaguar_wheel wheel_prefix="rear_left">
@@ -83,5 +83,5 @@
     </xacro:jaguar_wheel>
     <xacro:jaguar_wheel wheel_prefix="rear_right">
-        <origin xyz="${-wheelbase/2} ${-track/2} ${wheel_vertical_offset}" rpy="0 0 ${M_PI}"/>
+        <origin xyz="${-wheelbase/2} ${-track/2} ${wheel_vertical_offset}" rpy="0 0 0"/>
     </xacro:jaguar_wheel>
     <!-- Laser -->

Commit message: Update the robot description for better simulation

File: jaguar_description/urdf/jaguar.urdf.xacro (robot description, xacro)
@@ -92,5 +92,7 @@
     </joint>
     <link name="laser_link">
-        <visual>
+        <!-- Removing the laser visual and collision properties
+        because they affect the simulated pointcloud -->
+        <!--<visual>
             <origin xyz="0 0 0" rpy="0 0 0"/>
             <geometry>
@@ -100,11 +102,11 @@
                 <color rgba="0 0 255 0.8"/>
             </material>
-        </visual>
-        <collision>
+        </visual>-->
+        <!--<collision>
             <origin xyz="0 0 0" rpy="0 0 0"/>
             <geometry>
                 <box size="${laser_x_size} ${laser_y_size} ${laser_z_size}"/>
             </geometry>
-        </collision>
+        </collision>-->
     </link>
     <!-- Camera -->
@@ -127,5 +129,27 @@
             <origin xyz="0 0 0" rpy="0 ${M_PI/2} 0"/>
             <geometry>
-                <cylinder length="0.1" radius="${0.025/2}"/>
+                <cylinder length="${camera_length}" radius="${camera_radius}"/>
+            </geometry>
+        </collision>
+    </link>
+    <joint name="depth_camera_pole_joint" type="fixed">
+        <origin xyz="0 0 0.38" rpy="0 0 0"/>
+        <parent link="base_link"/>
+        <child link="depth_camera_pole_link"/>
+    </joint>
+    <link name="depth_camera_pole_link">
+        <visual>
+            <origin xyz="0 0 0" rpy="0 0 0"/>
+            <geometry>
+                <cylinder length="0.2625" radius="0.015"/>
+            </geometry>
+            <material name="black">
+                <color rgba="0 0 0 1"/>
+            </material>
+        </visual>
+        <collision>
+            <origin xyz="0 0 0" rpy="0 0 0"/>
+            <geometry>
+                <cylinder length="0.2625" radius="0.015"/>
             </geometry>
         </collision>

Commit message: Extra files and changes to introduce support for the Rubedos Viper stereo camera

File: jaguar_description/urdf/jaguar.urdf.xacro (robot description, xacro)
@@ -146,4 +146,22 @@
       <xacro:depth_camera prefix="camera"/>
     </xacro:if>
+    <xacro:if value="$(arg viper)">
+    <link name="camera_link">
+        <visual>
+            <origin xyz="0 0 0" rpy="${pi/2} 0 ${pi/2}"/>
+            <geometry>
+                <mesh filename="package://jaguar_description/meshes/CVM_Assembly_v4.0.1_RC27_shell.STL" scale="0.001 0.001 0.001"/>
+            </geometry>
+            <material name="black">
+                <color rgba="0.1 0.1 0.1 1.0"/>
+            </material>
+        </visual>
+    </link>
+     <joint name="camera_frame_joint" type="fixed">
+        <origin xyz="0 -0.125 0.525" rpy="0 0 0 "/>
+        <parent link="base_link"/>
+        <child link="camera_link"/>
+      </joint>
+    </xacro:if>
       <gazebo>
     <plugin name="gazebo_ros_control" filename="libgazebo_ros_control.so">

Commit message: Various fixes on the URDF. Accurate GPS position and better camera placement

File: jaguar_description/urdf/jaguar.urdf.xacro (robot description, xacro)
@@ -34,4 +34,15 @@
     <property name="camera_radius" value="${0.025/2}"/>
     <property name="camera_length" value="0.01"/>
+    <!-- Stereo cam mounting pole -->
+    <property name="pole_length" value="0.245"/>
+    <property name="pole_radius" value="0.03"/>
+    <!-- GPS mounting pole -->
+    <property name="gps_pole_length" value="0.155"/>
+    <property name="gps_pole_radius" value="0.02"/>
+    <property name="gps_pole_x" value="${-base_x_size/2+0.04}"/>
+    <property name="gps_pole_y" value="${base_y_size/2-0.04}"/>
+    <property name="gps_pole_z" value="${base_z_size+distance_from_ground+gps_pole_length/2}"/>
+    <property name="gps_top_plate_length" value="0.01"/>
+    <property name="gps_top_plate_radius" value="0.03"/>
     <!-- Base link is the center of the robot's bottom plate -->
     <link name="base_link">
@@ -94,19 +105,19 @@
         <!-- Removing the laser visual and collision properties
         because they affect the simulated pointcloud -->
-        <!--<visual>
+        <visual>
             <origin xyz="0 0 0" rpy="0 0 0"/>
             <geometry>
                 <box size="${laser_x_size} ${laser_y_size} ${laser_z_size}"/>
             </geometry>
-            <material name="blue">
-                <color rgba="0 0 255 0.8"/>
-            </material>
-        </visual>-->
-        <!--<collision>
+            <material name="black">
+                <color rgba="0 0 0 0.8"/>
+            </material>
+        </visual>
+        <collision>
             <origin xyz="0 0 0" rpy="0 0 0"/>
             <geometry>
                 <box size="${laser_x_size} ${laser_y_size} ${laser_z_size}"/>
             </geometry>
-        </collision>-->
+        </collision>
     </link>
     <!-- Camera -->
@@ -134,5 +145,5 @@
     </link>
     <joint name="depth_camera_pole_joint" type="fixed">
-        <origin xyz="0 0 0.38" rpy="0 0 0"/>
+        <origin xyz="0 0 ${base_z_size+distance_from_ground+pole_length/2}" rpy="0 0 0"/>
         <parent link="base_link"/>
         <child link="depth_camera_pole_link"/>
@@ -142,5 +153,5 @@
             <origin xyz="0 0 0" rpy="0 0 0"/>
             <geometry>
-                <cylinder length="0.2625" radius="0.015"/>
+                <cylinder length="${pole_length}" radius="${pole_radius}"/>
             </geometry>
             <material name="black">
@@ -151,12 +162,55 @@
             <origin xyz="0 0 0" rpy="0 0 0"/>
             <geometry>
-                <cylinder length="0.2625" radius="0.015"/>
-            </geometry>
-        </collision>
-    </link>
-    <!-- GPS exact position is unnecessary thus placed at the center of the platform. -->
+                <cylinder length="${pole_length}" radius="${pole_radius}"/>
+            </geometry>
+        </collision>
+    </link>
+    <joint name="gps_pole_joint" type="fixed">
+        <origin xyz="${gps_pole_x} ${gps_pole_y} ${gps_pole_z}" rpy="0 0 0"/>
+        <parent link="base_link"/>
+        <child link="gps_pole_link"/>
+    </joint>
+    <link name="gps_pole_link">
+        <visual>
+            <origin xyz="0 0 0" rpy="0 0 0"/>
+            <geometry>
+                <cylinder length="${gps_pole_length}" radius="${gps_pole_radius}"/>
+            </geometry>
+            <material name="black">
+                <color rgba="0 0 0 1"/>
+            </material>
+        </visual>
+        <collision>
+            <origin xyz="0 0 0" rpy="0 0 0"/>
+            <geometry>
+                <cylinder length="${gps_pole_length}" radius="${gps_pole_radius}"/>
+            </geometry>
+        </collision>
+    </link>
+    <link name="gps_top_plate_link">
+        <visual>
+            <origin xyz="0 0 0" rpy="0 0 0"/>
+            <geometry>
+                <cylinder length="${gps_top_plate_length}" radius="${gps_top_plate_radius}"/>
+            </geometry>
+            <material name="black">
+                <color rgba="0 0 0 1"/>
+            </material>
+        </visual>
+        <collision>
+            <origin xyz="0 0 0" rpy="0 0 0"/>
+            <geometry>
+                <cylinder length="${gps_top_plate_length}" radius="${gps_top_plate_radius}"/>
+            </geometry>
+        </collision>
+    </link>
+    <joint name="gps_top_plate_joint" type="fixed">
+        <origin xyz="0 0 ${gps_pole_length/2+gps_top_plate_length/2}" rpy="0 0 0"/>
+        <parent link="gps_pole_link"/>
+        <child link="gps_top_plate_link"/>
+    </joint>
     <joint name="gps_joint" type="fixed">
-        <origin xyz="0 0 ${base_z_size}" rpy="0 0 0"/>
-        <parent link="base_link"/>
+        <origin xyz="0 0 0" rpy="0 0 0"/>
+        <parent link="gps_top_plate_link"/>
         <child link="gps_link"/>
     </joint>
@@ -183,6 +237,6 @@
     </link>
      <joint name="camera_frame_joint" type="fixed">
-        <origin xyz="0 -0.125 0.525" rpy="0 0 0 "/>
-        <parent link="base_link"/>
+        <origin xyz="0 0 ${pole_length/2+0.015}" rpy="0 0 0"/>
+        <parent link="depth_camera_pole_link"/>
         <child link="camera_link"/>
       </joint>
